File: PCB/LP_MotherBoard_v1/lilypad_V2.sch (EAGLE design)
At the start: 27 parts, among them U1 INA169QPWRQ1PW8-M, X4 BQ24074

Commit message: update board schematic
Parts:
- removed C1: 0.1µF, adafruit:C-USC0805K
- removed R3: 10K, adafruit:R-US_M0805
- removed R5: 0.1/1%, resistor-shunt:SMT-REF
- removed U1: INA169QPWRQ1PW8-M, INA169-SOP8:INA169QPWRQ1PW8-M
Connections:
- removed net TMP_PRB: HP1.16, JP7.2, R12.2
- net A1: no longer R3.1, U1.OUT
- net CHARGER_IN: no longer R5.1, U1.VIN+
- net GND: now also JP9.2; no longer C1.2, R3.2, R5.2, U1.GND, U1.VIN-
- net P11: now also JP7.2, R12.2
- net VCC: no longer C1.1, U1.V-
Other:
- note removed: "Solar Hookup"
- moved on the sheet: JP9
